File: hardware/cdf-1/cdf-1.sch (KiCad schematic (older format))
At the start: 0 parts

Commit message: 1st prototype
Parts:
- added C2, C? (x15): C, symbol Device:C
- added C? (x3): CP, symbol Device:CP
- added D1: 3.3V POWER LED, symbol Device:LED
- added D2: DUT POWER CTRL LED, symbol Device:LED
- added D3: SPI PROG LED, symbol Device:LED
- added D4: DUT FETH LED, symbol Device:LED
- added D?: SPI DUT LED, symbol Device:LED
- added D?: WIFI LED, symbol Device:LED
- added D? (x2): LED, symbol Device:LED
- added FB?: Ferrite_Bead, symbol Device:Ferrite_Bead
- added J1: DUT SPI FLASH, symbol Connector_Generic:Conn_02x04_Counter_Clockwise
- added J3: SPI FLASH, symbol Connector_Generic:Conn_02x04_Counter_Clockwise
- added J4: DUT FETH, symbol Connector_Generic:Conn_01x04
- added J5: DUT POWER, symbol Connector_Generic:Conn_01x02
- added J6: DEBUG UART PROBE, symbol Connector_Generic:Conn_01x03
- added J?: DUT DC POWER IN, symbol Connector:Jack-DC
- added J?: 3.3V SOURCE, symbol Connector_Generic:Conn_01x03
- added J?: JUMPER STORAGE, symbol Connector_Generic:Conn_02x05_Counter_Clockwise
- added J?: WAN, symbol Connector:RJ45_LED
- added J?: FORCE USB POWER, symbol Connector_Generic:Conn_01x02
- added J?: DUT USB, symbol Connector_Generic:Conn_01x04
- added J?: FORCE PROG, symbol Connector_Generic:Conn_01x02
- added J?: I2C PROBE, symbol Connector_Generic:Conn_01x03
- added J?: SELF PROG, symbol Connector_Generic:Conn_01x03
- added J?: DUT UART, symbol Connector_Generic:Conn_01x03
- added J?: DUT UART PROBE, symbol Connector_Generic:Conn_01x03
- added J?: DUT POWER ON FORCE, symbol Connector_Generic:Conn_01x02
- added J?: FORCE RESET, symbol Connector_Generic:Conn_01x02
- added J?: SELF PROG OLD, symbol Connector_Generic:Conn_02x04_Counter_Clockwise
- added J?: MT7688 USB HOST, symbol Connector:USB_A
- added J?: DUT USB PORT, symbol Connector:USB_A
- added J?: DUT SPI FLASH PW SELECTOR, symbol Connector_Generic:Conn_01x03
- added J?: USB DEBUG, symbol Connector:USB_B_Micro
- added M1: hlk-7688a(mt7688), symbol components0:hlk-7688a(mt7688)
- added Q? (x3): BC847, Package_TO_SOT_SMD:SOT-23, symbol Transistor_BJT:BC847
- added Q? (x2): IRLML6402, Package_TO_SOT_SMD:SOT-23, symbol Transistor_FET:IRLML6402
- added Q? (x2): BC857, Package_TO_SOT_SMD:SOT-23, symbol Transistor_BJT:BC857
- added R10, R11, R3, R4, R5, R7, R8, R9, R? (x25): R, symbol Device:R
- added SW1: Encoder w BTN, symbol Device:Rotary_Encoder_Switch
- added SW2: RESET, symbol Switch:SW_MEC_5E
- added SW3: DUT POWER OFF, symbol Switch:SW_MEC_5E
- added U1: oled display(ssd1306), symbol components0:ssd1306
- added U2: INA219AxDCN, Package_TO_SOT_SMD:SOT-23-8, symbol Analog_ADC:INA219AxDCN
- added U3, U4: SN74CB3Q3257, symbol components0:SN74CB3Q3257
- added U?: LM1117GS-3.3, symbol Regulator_Linear:LM1117-3.3
- added U?: FT232RL, Package_SO:SSOP-28_5.3x10.2mm_P0.65mm, symbol Interface_USB:FT232RL
Connections:
- new net: M1.33 (WLED_N/GPIO44), R?.2
- new net: D2.2 (A), R?.2
- new net: D3.1 (K), Q?.3 (C)
- new net: D3.2 (A), R?.2
- new net: Q?.2 (S), R7.1, U2.1 (IN+)
- new net: J5.2 (Pin_2), R7.2, U2.2 (IN-)
- new net: R10.2, R8.1, U2.7 (A0)
- new net: R11.2, R9.1, U2.8 (A1)
- new net: R?.1, R?.2, U1.15 (D/C#)
- new net: C?.1, U1.2 (C2P)
- new net: R?.2, U1.26 (IREF)
- new net: C?.2, U1.27 (VCOMH)
- new net: C?.2, C?.2, U1.28 (VCC)
- new net: C?.2, U1.3 (C2N)
- new net: C?.1, U1.4 (C1P)
- new net: C?.2, U1.5 (C2N)
- new net: Q?.1 (B), R?.1 (x5)
- new net: Q?.3 (C), R?.2 (x3)
- new net: J?.1 (Pin_1), Q?.1 (G)
- new net: R?.1, R?.1, R?.2
- new net: J?.2 (Pin_2), U?.3 (VI)
- new net: R?.2, U3.3 (1B2)
- new net: R?.2, U3.6 (2B2)
- new net: D?.2 (A), Q?.3 (C)
- new net: D?.1 (K), R?.2
- new net: C?.2, U?.17 (3V3OUT), U?.20 (VCC)
- new net: R?.1, R?.2
- new net: J?.3 (D+), U?.15 (USBD+)
- new net: J?.2 (D-), U?.16 (USBD-)
- new net: R?.2, U?.22 (CBUS1)
- new net: R?.2, U?.23 (CBUS0)
- new net: D?.2 (A), R?.1
- new net: D?.1 (K), R?.1 (x2)
- new net +3V3: C2.2, C?.1, C?.1, C?.1, D?.2 (A), D?.2 (A), J?.3 (Pin_3), M1.2 (3.3V), M1.3 (3.3V), R10.1, R11.1, R3.2, R4.1, R5.1, R?.1, R?.1, R?.1, R?.1, R?.2, R?.2, U1.11 (BS1), U1.6 (VBAT), U1.9 (VDD), U2.4 (VS), U?.2 (VO)
- new net +5V: J?.1 (Pin_1), Q?.2 (S)
- new net DUT_POWER_CONTROL: R?.1, R?.2, SW3.3 (K), SW3.4 (A)
- new net DUT_SPI_CS: J1.1 (Pin_1), U4.2 (1B1)
- new net DUT_SPI_HOLD: J1.7 (Pin_7), U3.2 (1B1)
- new net DUT_SPI_MISO: J1.2 (Pin_2), U4.13 (4B2), U4.14 (4B1)
- new net DUT_SPI_MOSI: J1.5 (Pin_5), U4.10 (3B2)
- new net DUT_SPI_SCK: J1.6 (Pin_6), U4.5 (2B1)
- new net DUT_SPI_VCC: J1.8 (Pin_8), J?.1 (Pin_1)
- new net DUT_SPI_WP: J1.3 (Pin_3), U3.5 (2B1)
- new net GND: C2.1, C?.1, C?.1, C?.1, C?.1, C?.1, C?.1, C?.2, C?.2, C?.2, C?.2, C?.2, C?.2, C?.2, D2.1 (K), D?.1 (K), J1.4 (Pin_4), J3.4 (Pin_4), J5.1 (Pin_1), J6.1 (Pin_1), J?.1 (Pin_1), J?.1 (Pin_1), J?.2 (Pin_2), J?.2 (Pin_2), J?.3 (Pin_3), J?.4 (Pin_4), J?.5 (GND), J?.6 (Shield), M1.1 (GND), M1.21 (GND), M1.23 (GND), M1.4 (GND), M1.56 (GND), Q?.2 (E), Q?.2 (E), Q?.2 (E), R8.2, R9.2, R?.1, R?.1, R?.1, R?.2, R?.2, R?.2, SW1.C, SW1.S2, SW2.1, SW2.2, SW3.1, SW3.2, U1.10 (BS0), U1.12 (BS2), U1.13 (CS#), U1.16 (R/W#), U1.17 (E/RS#), U1.21 (D3), U1.22 (D4), U1.23 (D5), U1.24 (D6), U1.25 (D7), U1.29 (VLSS), U1.8 (VSS), U2.3 (GND), U3.10 (3B2), U3.11 (3B1), U3.12 (4A), U3.13 (4B2), U3.14 (4B1), U3.15 (/OE), U3.8 (GND), U3.9 (3A), U4.15 (/OE), U4.8 (GND), U?.1 (GND), U?.18 (GND), U?.21 (GND), U?.25 (AGND), U?.26 (TEST), U?.7 (GND)
- new net GND1: J?.1 (Pin_1), J?.10 (Pin_10), J?.2 (Pin_2), J?.3 (Pin_3), J?.4 (Pin_4), J?.5 (Pin_5), J?.6 (Pin_6), J?.7 (Pin_7), J?.8 (Pin_8), J?.9 (Pin_9)
- new net I2C_SCK: J?.2 (Pin_2), M1.24 (I2C_SCLK/GPIO04), R?.1
- new net I2C_SCL: U1.18 (D0), U2.5 (SCL)
- new net I2C_SDA: J?.1 (Pin_1), M1.25 (I2C_SD/GPIO05), R?.2, U1.19 (D1), U1.20 (D2), U2.6 (SDA)
- new net PROG_SPI_CS: J?.2 (Pin_2), U4.3 (1B2)
- new net PROG_SPI_CS0: J?.1 (Pin_1), J?.3 (Pin_3), M1.5 (SPI_CS0)
- new net PROG_SPI_CS1: J?.1 (Pin_1), M1.26 (SPI_CS1/GPIO06)
- new net PROG_SPI_MISO: J?.2 (Pin_2), M1.28 (SPI_MISO/GPIO09)
- new net PROG_SPI_MOSI: J?.5 (Pin_5), M1.29 (SPI_MOSI/GPIO08), U4.11 (3B1)
- new net PROG_SPI_SCK: J?.6 (Pin_6), M1.27 (SPI_CLK/GPIO07), U4.6 (2B2)
- new net PROG_SPI_WP: J?.3 (Pin_3)
- new net PRO_SPI_HOLD: J?.7 (Pin_7)
- new net RESET: J?.1 (Pin_1), M1.14 (PORST_N), SW2.3 (K), SW2.4 (A), U1.14 (RES#)
- new net SPI_CS: J3.1 (Pin_1), U4.4 (1A)
- new net SPI_HOLD: J3.7 (Pin_7), U3.4 (1A)
- new net SPI_MISO: J3.2 (Pin_2), U4.12 (4A)
- new net SPI_MOSI: J3.5 (Pin_5), U4.9 (3A)
- new net SPI_MUX_CONTROL: J?.2 (Pin_2), M1.30 (GPIO11), R?.1, R?.2, R?.2, U3.1 (Select), U4.1 (Select)
- new net SPI_SCK: J3.6 (Pin_6), U4.7 (2A)
- new net SPI_VCC: C?.1, C?.1, C?.1, C?.1, C?.2, C?.2, J3.8 (Pin_8), J?.1 (Pin_1), J?.2 (Pin_2), Q?.2 (E), R?.1, U3.16 (VCC), U4.16 (VCC)
- new net SPI_WP: J3.3 (Pin_3), U3.7 (2A)
- new net SW1_BUTTON: M1.9 (EPHY_LED4/JTAG_RST_N/GPIO39), R5.2, SW1.S1
- new net SW1_RA: M1.10 (EPHY_LED3/JTAG_CLK/GPIO40), R3.1, SW1.A
- new net SW1_RB: M1.11 (EPHY_LED2/JTAG_TMS/GPIO41), R4.2, SW1.B
- new net UART_DEBUG_RX: J6.2 (Pin_2), M1.32 (UART_RXD0/GPIO13), U?.1 (TXD)
- new net UART_DEBUG_TX: J6.3 (Pin_3), M1.31 (UART_TXD0/GPIO12), U?.5 (RXD)
- new net UART_DUT_RX: J?.2 (Pin_2), J?.2 (Pin_2), M1.16 (UART_RXD1/PWM1/GPIO46)
- new net UART_DUT_TX: J?.3 (Pin_3), J?.3 (Pin_3), M1.15 (UART_TXD1/PWM0/GPIO45)
- new net VBUS: J?.1 (VBUS), Q?.3 (D), R?.1
- new net VCC: J?.3 (Pin_3), Q?.2 (E), Q?.3 (D), R?.1
