File: hardware/cdf-2/debug.kicad_sch (KiCad schematic)
At the start: 0 parts

Commit message: improve
Parts:
- added D1, D2: LED, symbol Device:LED
- added J1: USB_B_Micro, symbol Connector:USB_B_Micro
- added R1, R2: R, symbol Device:R
- added U1: FT232RL, Package_SO:SSOP-28_5.3x10.2mm_P0.65mm, symbol Interface_USB:FT232RL
Connections:
- net GND: now also U1.18 (GND), U1.21 (GND), U1.25 (AGND), U1.7 (GND)
- new net: D2.1 (K), R2.1
- new net: D1.1 (K), R1.1
- no-connect marks 0 -> 9
Other:
- note added: "Host DEBUG"
Changed lines of the file:
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@@
 (kicad_sch (version 20210621) (generator eeschema)
   (paper "A4" portrait)
-  (hierarchical_label "UART_TX" (shape output) (at 48.26 36.83 0)
-    (effects (font (size 1.27 1.27)) (justify left))
+  (junction (at 77.47 138.43) (diameter 0) (color 0 0 0 0))
+  (junction (at 80.01 138.43) (diameter 0) (color 0 0 0 0))
+  (no_connect (at 97.79 100.33))
+  (no_connect (at 97.79 102.87))
+  (no_connect (at 97.79 105.41))
+  (no_connect (at 97.79 107.95))
+  (no_connect (at 97.79 110.49))
+  (no_connect (at 97.79 113.03))
+  (no_connect (at 97.79 125.73))
+  (no_connect (at 97.79 128.27))
+  (no_connect (at 97.79 130.81))
+  (wire (pts (xy 72.39 138.43) (xy 77.47 138.43))
+    (stroke (width 0) (type default) (color 0 0 0 0))
   )
-  (hierarchical_label "UART_RX" (shape input) (at 48.26 41.91 0)
-    (effects (font (size 1.27 1.27)) (justify left))
+  (wire (pts (xy 77.47 138.43) (xy 77.47 143.51))
+    (stroke (width 0) (type default) (color 0 0 0 0))
+  )
+  (wire (pts (xy 77.47 138.43) (xy 80.01 138.43))
+    (stroke (width 0) (type default) (color 0 0 0 0))
+  )
+  (wire (pts (xy 80.01 138.43) (xy 82.55 138.43))
+    (stroke (width 0) (type default) (color 0 0 0 0))
+  )
+  (text "Host DEBUG" (at 15.24 27.94 0)
+    (effects (font (size 8 8)) (justify left bottom))
   )
   (hierarchical_label "GND" (shape output) (at 48.26 58.42 0)
     (effects (font (size 1.27 1.27)) (justify left))
   )
+  (hierarchical_label "GND" (shape output) (at 77.47 143.51 270)
+    (effects (font (size 1.27 1.27)) (justify right))
+  )
+  (hierarchical_label "UART_TX" (shape output) (at 95.25 82.55 0)
+    (effects (font (size 1.27 1.27)) (justify left))
+  )
+  (hierarchical_label "UART_RX" (shape input) (at 95.25 85.09 0)
+    (effects (font (size 1.27 1.27)) (justify left))
+  )
+  (symbol (lib_id "Device:R") (at 111.76 104.14 0) (unit 1)
+    (in_bom yes) (on_board yes)
+    (property "Reference" "R1" (id 0) (at 113.538 103.2315 0)
+      (effects (font (size 1.27 1.27)) (justify left))
+    )
+    (property "Value" "R" (id 1) (at 113.538 106.0066 0)
+      (effects (font (size 1.27 1.27)) (justify left))
+    )
+    (property "Footprint" "" (id 2) (at 109.982 104.14 90)
+      (effects (font (size 1.27 1.27)) hide)
+    )
+    (property "Datasheet" "~" (id 3) (at 111.76 104.14 0)
+      (effects (font (size 1.27 1.27)) hide)
+    )
+    (pin "1")
+    (pin "2")
+  )
+  (symbol (lib_id "Device:R") (at 121.92 104.14 0) (unit 1)
+    (in_bom yes) (on_board yes) (fields_autoplaced)
+    (property "Reference" "R2" (id 0) (at 123.698 103.2315 0)
+      (effects (font (size 1.27 1.27)) (justify left))
+    )
+    (property "Value" "R" (id 1) (at 123.698 106.0066 0)
+      (effects (font (size 1.27 1.27)) (justify left))
+    )
+    (property "Footprint" "" (id 2) (at 120.142 104.14 90)
+      (effects (font (size 1.27 1.27)) hide)
+    )
+    (property "Datasheet" "~" (id 3) (at 121.92 104.14 0)
+      (effects (font (size 1.27 1.27)) hide)
+    )
+    (pin "1")
+    (pin "2")
+  )
+  (symbol (lib_id "Device:LED") (at 111.76 96.52 90) (unit 1)
+    (in_bom yes) (on_board yes) (fields_autoplaced)
+    (property "Reference" "D1" (id 0) (at 114.681 95.9924 90)
+      (effects (font (size 1.27 1.27)) (justify right))
+    )
+    (property "Value" "LED" (id 1) (at 114.681 98.7675 90)
+      (effects (font (size 1.27 1.27)) (justify right))
+    )
+    (property "Footprint" "" (id 2) (at 111.76 96.52 0)
+      (effects (font (size 1.27 1.27)) hide)
+    )
+    (property "Datasheet" "~" (id 3) (at 111.76 96.52 0)
+      (effects (font (size 1.27 1.27)) hide)
+    )
+    (pin "1")
+    (pin "2")
+  )
+  (symbol (lib_id "Device:LED") (at 121.92 96.52 90) (unit 1)
+    (in_bom yes) (on_board yes) (fields_autoplaced)
+    (property "Reference" "D2" (id 0) (at 124.841 95.9924 90)
+      (effects (font (size 1.27 1.27)) (justify right))
+    )
+    (property "Value" "LED" (id 1) (at 124.841 98.7675 90)
+      (effects (font (size 1.27 1.27)) (justify right))
+    )
+    (property "Footprint" "" (id 2) (at 121.92 96.52 0)
+      (effects (font (size 1.27 1.27)) hide)
+    )
+    (property "Datasheet" "~" (id 3) (at 121.92 96.52 0)
+      (effects (font (size 1.27 1.27)) hide)
+    )
+    (pin "1")
+    (pin "2")
+  )
+  (symbol (lib_id "Connector:USB_B_Micro") (at 30.48 99.06 0) (unit 1)
+    (in_bom yes) (on_board yes) (fields_autoplaced)
+    (property "Reference" "J1" (id 0) (at 31.6865 87.4734 0))
+    (property "Value" "USB_B_Micro" (id 1) (at 31.6865 90.2485 0))
+    (property "Footprint" "" (id 2) (at 34.29 100.33 0)
+      (effects (font (size 1.27 1.27)) hide)
+    )
+    (property "Datasheet" "~" (id 3) (at 34.29 100.33 0)
+      (effects (font (size 1.27 1.27)) hide)
+    )
+    (pin "1")
+    (pin "2")
+    (pin "3")
+    (pin "4")
+    (pin "5")
+    (pin "6")
+  )
+  (symbol (lib_id "Interface_USB:FT232RL") (at 77.47 113.03 0) (unit 1)
+    (in_bom yes) (on_board yes) (fields_autoplaced)
+    (property "Reference" "U1" (id 0) (at 77.47 83.7904 0))
+    (property "Value" "FT232RL" (id 1) (at 77.47 86.5655 0))
+    (property "Footprint" "Package_SO:SSOP-28_5.3x10.2mm_P0.65mm" (id 2) (at 105.41 135.89 0)
+      (effects (font (size 1.27 1.27)) hide)
+    )
+    (property "Datasheet" "https://www.ftdichip.com/Support/Documents/DataSheets/ICs/DS_FT232R.pdf" (id 3) (at 77.47 113.03 0)
+      (effects (font (size 1.27 1.27)) hide)
+    )
+    (pin "1")
+    (pin "10")
+    (pin "11")
+    (pin "12")
+    (pin "13")
+    (pin "14")
+    (pin "15")
+    (pin "16")
+    (pin "17")
+    (pin "18")
+    (pin "19")
+    (pin "2")
+    (pin "20")
+    (pin "21")
+    (pin "22")
+    (pin "23")
+    (pin "25")
+    (pin "26")
+    (pin "27")
+    (pin "28")
+    (pin "3")
+    (pin "4")
+    (pin "5")
+    (pin "6")
+    (pin "7")
+    (pin "9")
+  )
 )

Commit message: improve
Other:
- title: (none) -> Camera Debug Facility
Changed lines of the file:
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@@
 (kicad_sch (version 20210621) (generator eeschema)
   (paper "A4" portrait)
+  (title_block
+    (title "Camera Debug Facility")
+    (date "2021-10-31")
+    (rev "2.1.0-pre1")
+  )
   (junction (at 77.47 138.43) (diameter 0) (color 0 0 0 0))
   (junction (at 80.01 138.43) (diameter 0) (color 0 0 0 0))
