File: hardware/cdf-2/power.kicad_sch (KiCad schematic)
At the start: 0 parts

Commit message: improve
Other:
- title: (none) -> Camera Debug Facility
Changed lines of the file:
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@@
 (kicad_sch (version 20210621) (generator eeschema)
   (paper "A4" portrait)
+  (title_block
+    (title "Camera Debug Facility")
+    (date "2021-10-31")
+    (rev "2.1.0-pre1")
+  )
   (hierarchical_label "12V" (shape output) (at 59.69 48.26 0)
     (effects (font (size 1.27 1.27)) (justify left))
