File: hardware/cdf-2/spi_muxer.kicad_sch (KiCad schematic)
At the start: 0 parts

Commit message: improve
Parts:
- added J?: Conn_02x04_Counter_Clockwise, Package_DIP:DIP-8_W7.62mm_Socket_LongPads, symbol Connector_Generic:Conn_02x04_Counter_Clockwise
- added U? (x2): SN74CB3Q3257, symbol components0:SN74CB3Q3257
Other:
- title: (none) -> Camera Debug Facility
Changed lines of the file:
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@@
 (kicad_sch (version 20210621) (generator eeschema)
   (paper "A4" portrait)
+  (title_block
+    (title "Camera Debug Facility")
+    (date "2021-10-31")
+    (rev "2.1.0-pre1")
+  )
   (hierarchical_label "3.3V" (shape input) (at 39.37 44.45 0)
     (effects (font (size 1.27 1.27)) (justify left))
@@
     (effects (font (size 1.27 1.27)) (justify left))
   )
+  (symbol (lib_id "Connector_Generic:Conn_02x04_Counter_Clockwise") (at 105.41 76.2 0) (unit 1)
+    (in_bom yes) (on_board yes) (fields_autoplaced)
+    (property "Reference" "J?" (id 0) (at 106.68 68.4235 0))
+    (property "Value" "Conn_02x04_Counter_Clockwise" (id 1) (at 106.68 71.1986 0))
+    (property "Footprint" "Package_DIP:DIP-8_W7.62mm_Socket_LongPads" (id 2) (at 105.41 76.2 0)
+      (effects (font (size 1.27 1.27)) hide)
+    )
+    (property "Datasheet" "~" (id 3) (at 105.41 76.2 0)
+      (effects (font (size 1.27 1.27)) hide)
+    )
+    (pin "1")
+    (pin "2")
+    (pin "3")
+    (pin "4")
+    (pin "5")
+    (pin "6")
+    (pin "7")
+    (pin "8")
+  )
+  (symbol (lib_id "components0:SN74CB3Q3257") (at 78.74 111.76 0) (unit 1)
+    (in_bom yes) (on_board yes) (fields_autoplaced)
+    (property "Reference" "U?" (id 0) (at 78.74 96.4905 0))
+    (property "Value" "SN74CB3Q3257" (id 1) (at 78.74 99.2656 0))
+    (property "Footprint" "" (id 2) (at 80.01 99.06 0)
+      (effects (font (size 1.27 1.27)) hide)
+    )
+    (property "Datasheet" "" (id 3) (at 80.01 99.06 0)
+      (effects (font (size 1.27 1.27)) hide)
+    )
+    (pin "1")
+    (pin "10")
+    (pin "11")
+    (pin "12")
+    (pin "13")
+    (pin "14")
+    (pin "15")
+    (pin "16")
+    (pin "2")
+    (pin "3")
+    (pin "4")
+    (pin "5")
+    (pin "6")
+    (pin "7")
+    (pin "8")
+    (pin "9")
+  )
+  (symbol (lib_id "components0:SN74CB3Q3257") (at 80.01 147.32 0) (unit 1)
+    (in_bom yes) (on_board yes) (fields_autoplaced)
+    (property "Reference" "U?" (id 0) (at 80.01 132.0505 0))
+    (property "Value" "SN74CB3Q3257" (id 1) (at 80.01 134.8256 0))
+    (property "Footprint" "" (id 2) (at 81.28 134.62 0)
+      (effects (font (size 1.27 1.27)) hide)
+    )
+    (property "Datasheet" "" (id 3) (at 81.28 134.62 0)
+      (effects (font (size 1.27 1.27)) hide)
+    )
+    (pin "1")
+    (pin "10")
+    (pin "11")
+    (pin "12")
+    (pin "13")
+    (pin "14")
+    (pin "15")
+    (pin "16")
+    (pin "2")
+    (pin "3")
+    (pin "4")
+    (pin "5")
+    (pin "6")
+    (pin "7")
+    (pin "8")
+    (pin "9")
+  )
 )
