File: hardware/cdf-2/host.kicad_sch (KiCad schematic)
At the start: 0 parts

Commit message: improve
Other:
- title: (none) -> Camera Debug Facility
Changed lines of the file:
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@@
 (kicad_sch (version 20210621) (generator eeschema)
   (paper "A4" portrait)
+  (title_block
+    (title "Camera Debug Facility")
+    (date "2021-10-31")
+    (rev "2.1.0-pre1")
+  )
   (hierarchical_label "12V" (shape input) (at 43.18 35.56 0)
     (effects (font (size 1.27 1.27)) (justify left))

Commit message: improve
Parts:
- added C? (x2): C, Capacitor_SMD:C_0603_1608Metric, symbol Device:C
- added C? (x2): CP, Capacitor_Tantalum_SMD:CP_EIA-7343-31_Kemet-D_Pad2.25x2.55mm_HandSolder, symbol Device:CP
- added C? (x4): C, Capacitor_SMD:C_0805_2012Metric, symbol Device:C
- added D?: WIFI LED, LED_SMD:LED_0805_2012Metric, symbol Device:LED
- added D?: WAN LED, LED_SMD:LED_0805_2012Metric, symbol Device:LED
- added J?: WAN, Connector_RJ:RJ45_Amphenol_RJMG1BD3B8K1ANR, symbol components0:J00-0045NL
- added J?: MT7688 USB HOST, Connector_USB:USB_A_Molex_67643_Horizontal, symbol Connector:USB_A
- added J?: DUT FETH T, Connector_Molex:Molex_PicoBlade_53398-0471_1x04-1MP_P1.25mm_Vertical, symbol Connector_Generic:Conn_01x04
- added J?: DEBUG UART PROBE, Connector_PinHeader_2.54mm:PinHeader_1x03_P2.54mm_Vertical_SMD_Pin1Left, symbol Connector_Generic:Conn_01x03
- added J?: self prog, symbol Connector_Generic:Conn_02x04_Counter_Clockwise
- added JP?: VBUS SRC, Connector_PinHeader_2.54mm:PinHeader_2x03_P2.54mm_Vertical_SMD, symbol Connector_Generic:Conn_02x03_Odd_Even
- added JP?: FORCE RESET, Connector_PinHeader_2.54mm:PinHeader_1x02_P2.54mm_Vertical_SMD_Pin1Left, symbol Jumper:Jumper_2_Open
- added NT?: 3V3, symbol Device:NetTie_2
- added R? (x9): R, Resistor_SMD:R_0805_2012Metric, symbol Device:R
- added R? (x2): R, symbol Device:R
- added R?: 75, Resistor_SMD:R_0805_2012Metric, symbol Device:R
- added SW?: RESET, Button_Switch_SMD:SW_Push_1P1T_NO_6x6mm_H9.5mm, symbol Switch:SW_Push
- added U? (x2): EPCOS_A8065, Transformer_SMD:Transformer_Pulse_H1100NL, symbol components0:EPCOS_A8065
- added U? (x2): JS76x8, cdf-1:JS76x8, symbol components0:JS76x8
- added U?: LM1117-5.0, Package_TO_SOT_SMD:SOT-223-3_TabPin2, symbol Regulator_Linear:LM1117-5.0
Connections:
- net 3.3V: now also NT?.1, U?.3 (VDD3V3), U?.4 (VDD3V3)
- net ENCODER_A: now also U?.18 (EPHY_LED3_N_JTCLK)
- net ENCODER_B: now also U?.19 (EPHY_LED2_N_JTMS)
- net ENCODER_BTN: now also U?.17 (EPHY_LED4_N_JTRST_N)
- net GND: now also C?.1, C?.1, C?.1, C?.2, C?.2, C?.2, C?.2, C?.2, J?.3 (Pin_3), J?.4 (GND), J?.4 (Pin_4), J?.5 (Shield), J?.R7 (NC), J?.R8 (CHS_GROUND), JP?.1 (A), SW?.1, U?.1 (GND), U?.1 (GND), U?.1 (GND), U?.11 (GND), U?.11 (GND), U?.2 (GND), U?.23 (GND), U?.23 (GND), U?.26 (GND), U?.26 (GND), U?.29 (GND), U?.29 (GND), U?.32 (GND), U?.32 (GND), U?.36 (GND), U?.36 (GND), U?.45 (GND), U?.45 (GND), U?.5 (GND), U?.5 (GND), U?.50 (GND), U?.50 (GND), U?.55 (GND), U?.55 (GND), U?.60 (GND), U?.60 (GND), U?.65 (GND), U?.65 (GND), U?.70 (GND), U?.70 (GND), U?.73 (GND), U?.73 (GND), U?.8 (GND), U?.8 (GND)
- net I2C_CLK: now also R?.2, U?.33 (I2C_SCLK)
- net I2C_DAT: now also R?.1, U?.34 (I2C_SD)
- net LAN_R_N: now also U?.9 (RX-)
- net LAN_R_P: now also U?.11 (RX+)
- net LAN_T_N: now also U?.14 (TX-)
- net LAN_T_P: now also U?.16 (TX+)
- net MUX_CONTROL: now also U?.42 (GPIO11)
- net RESET: now also JP?.2 (B), R?.2, SW?.2, U?.14 (PERST_N)
- net SPI_CLK: now also J?.6 (Pin_6), U?.40 (SPI_CLK)
- net SPI_CS1: now also U?.37 (SPI_CS1)
- net SPI_MISO: now also J?.2 (Pin_2), U?.41 (SPI_MISO)
- net SPI_MOSI: now also J?.5 (Pin_5), U?.39 (SPI_MOSI)
- net UART1_RX: now also U?.25 (UART_RXD1)
- net UART1_TX: now also U?.24 (UART_TXD1)
- net UART_RX: now also U?.43 (UART_RXD0)
- net UART_TX: now also U?.44 (UART_TXD0)
- new net: D?.1 (K), R?.2
- new net: J?.L4, R?.2
- new net: C?.1, J?.R4 (CT), J?.R5 (CT)
- new net: U?.1 (TD+), U?.53 (MDI_R_P1_P)
- new net: U?.3 (TD-), U?.54 (MDI_R_P1_N)
- new net: U?.51 (MDI_T_P1_P), U?.6 (RD+)
- new net: U?.52 (MDI_T_P1_N), U?.8 (RD-)
- new net: J?.1 (VBUS), JP?.1 (Pin_1), JP?.3 (Pin_3), JP?.5 (Pin_5)
- new net: J?.1 (Pin_1), R?.1
- new net: C?.1, C?.1, JP?.6 (Pin_6), U?.2 (VO)
- new net: J?.2 (Pin_2), R?.1
- new net: R?.1, U?.22 (WLED_N)
- new net: C?.1, R?.2
- new net: R?.1, U?.10 (CT), U?.15 (CT)
- new net: U?.2 (CT), U?.7 (CT)
- new net: D?.2 (A), R?.2
- new net +3V3: D?.2 (A), R?.1, R?.1, R?.1, R?.1, R?.1, R?.2, U?.3 (VDD3V3)
- new net +5V: JP?.4 (Pin_4)
- new net 3V3_SIGNAL: NT?.2, R?.1, R?.2
- new net DUT_ETH_LED: U?.20 (EPHY_LED1_N_JTDI)
- new net DUT_ETH_R_N: U?.54 (MDI_R_P1_N), U?.8 (RD-)
- new net DUT_ETH_R_P: U?.53 (MDI_R_P1_P), U?.6 (RD+)
- new net DUT_ETH_T_N: U?.3 (TD-), U?.52 (MDI_T_P1_N)
- new net DUT_ETH_T_P: U?.1 (TD+), U?.51 (MDI_T_P1_P)
- new net DUT_POWER_CONTROL: U?.31 (I2S_CLK)
- new net DUT_T_ETH_R_N: J?.4 (Pin_4), U?.9 (RX-)
- new net DUT_T_ETH_R_P: J?.3 (Pin_3), U?.11 (RX+)
- new net DUT_T_ETH_T_N: J?.2 (Pin_2), U?.14 (TX-)
- new net DUT_T_ETH_T_P: J?.1 (Pin_1), U?.16 (TX+)
- new net HOST_SPI_CS0: J?.1 (Pin_1), U?.38 (SPI_CS0)
- new net HOST_SPI_HOLD: J?.7 (Pin_7)
- new net HOST_SPI_VCC: J?.8 (Pin_8), U?.35 (VDD3V3_PROG)
- new net HOST_SPI_WP: J?.3 (Pin_3)
- new net H_USB_N: J?.2 (D-), U?.72 (USB_N)
- new net H_USB_P: J?.3 (D+), U?.71 (USB_P)
- new net I2C_SCL: C?.1, R?.2, U?.33 (I2C_SCLK)
- new net I2C_SDA: C?.2, R?.1, U?.34 (I2C_SD)
- new net PROG_SPI_CS0: U?.38 (SPI_CS0)
- new net PROG_SPI_CS1: R?.2, U?.37 (SPI_CS1)
- new net PROG_SPI_MISO: U?.41 (SPI_MISO)
- new net PROG_SPI_MOSI: U?.39 (SPI_MOSI)
- new net PROG_SPI_SCK: U?.40 (SPI_CLK)
- new net SPI_MUXER_3V3_CONTROL: U?.28 (I2S_WS)
- new net SPI_MUX_CONTROL: U?.42 (GPIO11)
- new net SW_BUTTON: U?.17 (EPHY_LED4_N_JTRST_N)
- new net SW_RA: U?.18 (EPHY_LED3_N_JTCLK)
- new net SW_RB: U?.19 (EPHY_LED2_N_JTMS)
- new net UART_DEBUG_RX: R?.2, U?.44 (UART_TXD0)
- new net UART_DEBUG_TX: R?.2, U?.43 (UART_RXD0)
- new net UART_DUT_N: U?.25 (UART_RXD1)
- new net UART_DUT_P: U?.24 (UART_TXD1)
- new net VCC: C?.2, C?.2, JP?.2 (Pin_2), U?.3 (VI)
- new net WAN_LED: D?.1 (K), J?.L3, U?.21 (EPHY_LED0_N_JTDO)
- new net WAN_R_N: J?.R6 (RD-), U?.47 (MDI_R_P0_N)
- new net WAN_R_P: J?.R3 (RD+), U?.46 (MDI_R_P0_P)
- new net WAN_T_N: J?.R2 (TD-), U?.49 (MDI_T_P0_N)
- new net WAN_T_P: J?.R1 (TD+), U?.48 (MDI_T_P0_P)
- no-connect marks 0 -> 35
Other:
- note added: "ATTENTION! No overvoltage protection"
- note added: "J00-0045NL (same as HR911105A) RJ45 with embedded Trans."
- note added: "MT76x8 UNIT"
